Commit message: Adding IMU to the sensor list in the simulation

File: igvc_self_drive_description/urdf/gem_sensors.urdf.xacro (robot description, xacro)
@@ -3,14 +3,14 @@
   <xacro:property name="M_PI" value="3.1415926535897931" />
   <!-- Camera -->
-  <xacro:include filename="$(find igvc_self_drive_description)/urdf/sensors/camera.urdf.xacro" />
+  <!-- <xacro:include filename="$(find igvc_self_drive_description)/urdf/sensors/camera.urdf.xacro" />
   <xacro:camera_sim name="camera_front" parent="base_footprint" >
     <origin xyz="1.75 0 2.1" rpy="0 0.55 0" />
-  </xacro:camera_sim>
+  </xacro:camera_sim> -->
   <!-- LIDAR -->
-  <xacro:include filename="$(find hector_xacro_tools)/urdf/inertia_tensors.urdf.xacro" />
+  <!-- <xacro:include filename="$(find hector_xacro_tools)/urdf/inertia_tensors.urdf.xacro" />
   <xacro:include filename="$(find hector_sensors_description)/urdf/vlp16.urdf.xacro" />
   <xacro:vlp16 name="lidar" parent="base_footprint" ros_topic="/lidar">
     <origin xyz="2.75 0 0.85" rpy="0 0 0" />
-  </xacro:vlp16>
+  </xacro:vlp16> -->
   <!-- GPS -->
   <xacro:include filename="$(find igvc_self_drive_description)/urdf/sensors/gps.urdf.xacro" />
@@ -18,4 +18,28 @@
     <origin xyz="0.8 0 2.35" rpy="0 0 0" />
   </xacro:gps>
+  <!-- IMU -->
+  <xacro:include filename="$(find sensor_sim_gazebo)/urdf/imu.xacro" />
+  <xacro:imu name="imu" parent="base_footprint">
+    <origin xyz="1.0 0 2.35" rpy="0 0 0"/>
+  </xacro:imu>
+  <!-- <gazebo reference="imu_link">
+    <gravity>true</gravity>
+    <sensor name="imu_sensor" type="imu">
+      <always_on>true</always_on>
+      <update_rate>100</update_rate>
+      <visualize>true</visualize>
+      <topic>/imu</topic>
+      <plugin filename="libgazebo_ros_imu_sensor.so" name="imu_plugin">
+        <topicName>imu</topicName>
+        <bodyName>imu_link</bodyName>
+        <updateRateHZ>10.0</updateRateHZ>
+        <gaussianNoise>0.0</gaussianNoise>
+        <xyzOffset>0 0 0</xyzOffset>
+        <rpyOffset>0 0 0</rpyOffset>
+        <frameName>imu_link</frameName>
+      </plugin>
+      <pose>0 0 0 0 0 0</pose>
+    </sensor>
+  </gazebo> -->
   <!-- Sonar sensors -->
   <!-- <xacro:include filename="$(find hector_sensors_description)/urdf/sonar_sensor.urdf.xacro" />

Commit message: sensors for gazebo

File: igvc_self_drive_description/urdf/gem_sensors.urdf.xacro (robot description, xacro)
@@ -6,4 +6,8 @@
   <xacro:generic_camera name="camera_front" parent="base_footprint" ros_topic="/img" cam_info_topic="/cameraInfo" update_rate="10" res_x="640" res_y="480" image_format="R8G8B8" hfov="30">
     <origin xyz="1.75 0 2.1" rpy="0 0.55 0" />
+  </xacro:generic_camera>
+  <!-- Camera -->
+   <xacro:generic_camera name="camera_side" parent="base_footprint" ros_topic="/stop_camera" cam_info_topic="/cameraInfoStop" update_rate="10" res_x="640" res_y="480" image_format="R8G8B8" hfov="30">
+    <origin xyz="2 -.5 2.1" rpy="0 0 0" />
   </xacro:generic_camera>
   <!-- LIDAR -->
@@ -18,4 +22,12 @@
     <origin xyz="0.8 0 2.35" rpy="0 0 0" />
   </xacro:gps>
+  <!-- Realsense d435 -->
+  <!--     <xacro:macro name="realsense_d435_camera_gazebo_plugin_macro" params="name parent image_topic depth_points_topic min_range max_range update_rate"> -->
+  <xacro:include filename="$(find hector_sensors_description)/urdf/realsense_d435_camera.urdf.xacro" />
+  <xacro:realsense_d435_camera_model name="realsense" parent="base_footprint">
+      <origin xyz="2 0 1" rpy="0 0 0" />
+  </xacro:realsense_d435_camera_model>
+  <xacro:realsense_d435_camera_gazebo_plugin_macro parent="base_footprint" name="realsense" image_topic="/realsenseCam" depth_points_topic="/realsensepoints" min_range="0.01" max_range="100" update_rate="3" >
+  </xacro:realsense_d435_camera_gazebo_plugin_macro>
   <!-- IMU -->
   <xacro:include filename="$(find sensor_sim_gazebo)/urdf/imu.xacro" />
